File: demodulador_sicom/demodulador_sicom.kicad_sch (KiCad schematic)
At the start: 33 parts, among them J1 POWER, J2 OUTPUT, J3 CARRIER_IN, J4 SSB_IN, U1 MC1496D, U2 L7812

Commit message: Update pcb layout.
Parts:
- added H1, H2, H3: MountingHole, MountingHole:MountingHole_3.2mm_M3, symbol Mechanical:MountingHole
Other:
- company: (none) -> UTN - FRBB
- title: (none) -> Demodulador MC1496
- moved on the sheet: C1, C10, C11, C12, C13, C2, C3, C4, C5, C6, C7, C8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

Commit message: Fix missing connection.
- Add RP diode.
Parts:
- added D2: 1N4007, Diode_SMD:D_SMA_Handsoldering, symbol Diode:1N4007
Connections:
- net V_IN: now also D2.1 (K); no longer J1.1 (Pin_1)
- net at R3.2, U1.8 (IN_CARRIER): now also C5.1, R7.2, R8.2
- new net: D2.2 (A), J1.1 (Pin_1)
Changed lines of the file:
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@@
+	)
+	(junction
+		(at 113.03 107.95)
+		(diameter 0)
+		(color 0 0 0 0)
 	)
 	(junction
@@
 	)
 	(junction
-		(at 99.06 49.53)
-		(diameter 0)
-		(color 0 0 0 0)
-	)
-	(junction
 		(at 90.17 111.76)
 		(diameter 0)
@@
 	)
 	(junction
+		(at 99.06 49.53)
+		(diameter 0)
+		(color 0 0 0 0)
+	)
+	(junction
 		(at 114.3 113.03)
 		(diameter 0)
@@
 	(wire
 		(pts
+			(xy 80.01 49.53) (xy 87.63 49.53)
+		)
+		(stroke
+			(width 0)
+			(type default)
+		)
+	)
+	(wire
+		(pts
 			(xy 83.82 100.33) (xy 90.17 100.33)
 		)
@@
 	(wire
 		(pts
-			(xy 80.01 49.53) (xy 99.06 49.53)
-		)
-		(stroke
-			(width 0)
-			(type default)
-		)
-	)
-	(wire
-		(pts
 			(xy 171.45 97.79) (xy 168.91 97.79)
 		)
@@
 	(wire
 		(pts
+			(xy 104.14 107.95) (xy 113.03 107.95)
+		)
+		(stroke
+			(width 0)
+			(type default)
+		)
+	)
+	(wire
+		(pts
 			(xy 209.55 114.3) (xy 218.44 114.3)
 		)
@@
 	(wire
 		(pts
+			(xy 90.17 100.33) (xy 104.14 100.33)
+		)
+		(stroke
+			(width 0)
+			(type default)
+		)
+	)
+	(wire
+		(pts
+			(xy 104.14 100.33) (xy 104.14 107.95)
+		)
+		(stroke
+			(width 0)
+			(type default)
+		)
+	)
+	(wire
+		(pts
 			(xy 176.53 114.3) (xy 180.34 114.3)
 		)
@@
 		(pts
 			(xy 102.87 138.43) (xy 102.87 139.7)
+		)
+		(stroke
+			(width 0)
+			(type default)
+		)
+	)
+	(wire
+		(pts
+			(xy 95.25 49.53) (xy 99.06 49.53)
 		)
 		(stroke
@@
 	)
 	(symbol
+		(lib_id "Diode:1N4007")
+		(at 91.44 49.53 180)
+		(unit 1)
+		(exclude_from_sim no)
+		(in_bom yes)
+		(on_board yes)
+		(dnp no)
+		(fields_autoplaced yes)
+		(property "Reference" "D2"
+			(at 91.44 43.18 0)
+			(effects
+				(font
+					(size 1.27 1.27)
+				)
+			)
+		)
+		(property "Value" "1N4007"
+			(at 91.44 45.72 0)
+			(effects
+				(font
+					(size 1.27 1.27)
+				)
+			)
+		)
+		(property "Footprint" "Diode_SMD:D_SMA_Handsoldering"
+			(at 91.44 45.085 0)
+			(effects
+				(font
+					(size 1.27 1.27)
+				)
+				(hide yes)
+			)
+		)
+		(property "Datasheet" "http://www.vishay.com/docs/88503/1n4001.pdf"
+			(at 91.44 49.53 0)
+			(effects
+				(font
+					(size 1.27 1.27)
+				)
+				(hide yes)
+			)
+		)
+		(property "Description" "1000V 1A General Purpose Rectifier Diode, DO-41"
+			(at 91.44 49.53 0)
+			(effects
+				(font
+					(size 1.27 1.27)
+				)
+				(hide yes)
+			)
+		)
+		(property "Sim.Device" "D"
+			(at 91.44 49.53 0)
+			(effects
+				(font
+					(size 1.27 1.27)
+				)
+				(hide yes)
+			)
+		)
+		(property "Sim.Pins" "1=K 2=A"
+			(at 91.44 49.53 0)
+			(effects
+				(font
+					(size 1.27 1.27)
+				)
+				(hide yes)
+			)
+		)
+		(pin "2"
+		)
+		(pin "1"
+		)
+		(instances
+			(project ""
+				(path "/e67a33ca-5505-4c28-9d17-ef0bda0bd220"
+					(reference "D2")
+					(unit 1)
+				)
+			)
+		)
+	)
+	(symbol
 		(lib_id "Device:R")
 		(at 107.95 110.49 90)
@@
 		(dnp no)
 		(property "Reference" "R4"
-			(at 107.696 108.204 90)
-			(effects
-				(font
+			(at 103.124 109.474 90)
+			(effects
+				(font

Commit message: Change BNC footprint.
- Replace vias for holes, so they can have thermal relief.
- Export fabrication files
Parts:
- J2, J3, J4: footprint Connector_Coaxial:BNC_TEConnectivity_1478204_Vertical -> connector:BNC_TEConnectivity_413969-2
Other:
- added sheet Thermal reliefs vias (thermal_relief_vias.kicad_sch)
Changed lines of the file:
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@@
 			)
 		)
-		(property "Footprint" "Connector_Coaxial:BNC_TEConnectivity_1478204_Vertical"
+		(property "Footprint" "connector:BNC_TEConnectivity_413969-2"
 			(at 106.68 87.63 0)
 			(effects
@@
 			)
 		)
-		(property "Footprint" "Connector_Coaxial:BNC_TEConnectivity_1478204_Vertical"
+		(property "Footprint" "connector:BNC_TEConnectivity_413969-2"
 			(at 223.52 114.3 0)
 			(effects
@@
 			)
 		)
-		(property "Footprint" "Connector_Coaxial:BNC_TEConnectivity_1478204_Vertical"
+		(property "Footprint" "connector:BNC_TEConnectivity_413969-2"
 			(at 102.87 133.35 0)
 			(effects
@@
 				)
 			)
+		)
+	)
+	(sheet
+		(at 231.775 26.67)
+		(size 28.575 14.605)
+		(fields_autoplaced yes)
+		(stroke
+			(width 0.1524)
+			(type solid)
+		)
+		(fill
+			(color 0 0 0 0.0000)
+		)
+		(property "Sheetname" "Thermal reliefs vias"
+			(at 231.775 25.9584 0)
+			(effects
+				(font
+					(size 1.27 1.27)
+				)
+				(justify left bottom)
+			)
+		)
+		(property "Sheetfile" "thermal_relief_vias.kicad_sch"
+			(at 231.775 41.8596 0)
+			(effects
+				(font
+					(size 1.27 1.27)
+				)
+				(justify left top)
+			)
+		)
+		(instances
+			(project "demodulador_sicom"
+				(path "/e67a33ca-5505-4c28-9d17-ef0bda0bd220"
+					(page "2")
+				)
+			)
