File: modulador_sicom/modulador_sicom.kicad_sch (KiCad schematic)
At the start: 31 parts, among them J1 POWER, J2 OUTPUT, J3 CARRIER_IN, J4 SSB_IN, U1 MC1496D, U2 L7812

Commit message: Update pcb layout.
Parts:
- added C12: 25u, symbol Device:C_Polarized
- added C13: 100n, Inductor_SMD:L_1206_3216Metric_Pad1.42x1.75mm_HandSolder, symbol Device:C
Connections:
- net GND: now also C12.2, C13.2
- net at R3.2, U1.8 (IN_CARRIER): now also C12.1, C13.1
Other:
- moved on the sheet: C1, C11, C4, C5, J4, R4, R5, R6, R7, R8

Commit message: Update latest changes.
Parts:
- removed C1, C11, C2, C3, C4, C5: 100n, Inductor_SMD:L_1206_3216Metric_Pad1.42x1.75mm_HandSolder, symbol Device:C
- removed C8: 4.7n, Capacitor_SMD:C_0805_2012Metric_Pad1.18x1.45mm_HandSolder, symbol Device:C
- removed D1: LED, LED_THT:LED_D5.0mm, symbol Device:LED
- removed J1: POWER, Connector_PinHeader_2.54mm:PinHeader_1x02_P2.54mm_Vertical, symbol Connector:Conn_01x02_Pin
- removed R1, R11, R5: 1k, Resistor_SMD:R_0805_2012Metric_Pad1.20x1.40mm_HandSolder, symbol Device:R
- removed R13: 51, Resistor_SMD:R_0805_2012Metric_Pad1.20x1.40mm_HandSolder, symbol Device:R
- removed U2: L7812, Package_TO_SOT_SMD:TO-252-2, symbol Regulator_Linear:L7812
- added C1: 25u, Capacitor_THT:CP_Radial_D5.0mm_P2.50mm, symbol Device:C_Polarized
- added C4, C5, C8: 10u, Capacitor_THT:CP_Radial_D5.0mm_P2.50mm, symbol Device:C_Polarized
- added D2: 1N4007, Diode_SMD:D_SMA_Handsoldering, symbol Diode:1N4007
- added D3: LED, LED_THT:LED_D5.0mm, symbol Device:LED
- added H1, H2, H3: MountingHole, MountingHole:MountingHole_3.2mm_M3, symbol Mechanical:MountingHole
- added H4, H5: ~, via:Via_0.7x1.5, symbol vias:VIA
- added J5: POWER, Connector_PinHeader_2.54mm:PinHeader_1x02_P2.54mm_Vertical, symbol Connector:Conn_01x02_Pin
- added R14, R15: 100, Resistor_SMD:R_0805_2012Metric_Pad1.20x1.40mm_HandSolder, symbol Device:R
- added R16, R17: 10k, Resistor_SMD:R_0805_2012Metric_Pad1.20x1.40mm_HandSolder, symbol Device:R
- added RV1: 10k, Potentiometer_THT:Potentiometer_Bourns_3296W_Vertical, symbol Device:R_Potentiometer
- added U3: L7812, Package_TO_SOT_SMD:TO-252-2, symbol Regulator_Linear:L7812
- C12: footprint (none) -> Capacitor_THT:CP_Radial_D5.0mm_P2.50mm
- C6, C7: value 4.7n -> 100n; footprint Capacitor_SMD:C_0805_2012Metric_Pad1.18x1.45mm_HandSolder -> Inductor_SMD:L_1206_3216Metric_Pad1.42x1.75mm_HandSolder
- J2, J3: footprint (none) -> connector:BNC_TEConnectivity_413969-2
- J4: value SSB_IN -> MODULATING; footprint (none) -> connector:BNC_TEConnectivity_413969-2
- R2: value 51 -> 1k
Connections:
- net +12V: now also C7.1, R12.2, R2.1, C8.1, H5.1 (Via), U3.3 (OUT); no longer R12.1
- net GND: now also R6.2, C1.2, C5.2, C8.2, D3.1 (K), H4.1 (Via), J5.2 (Pin_2), RV1.2, U3.2 (GND); no longer R6.1
- net at C12.1, C13.1, R3.2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: now also R7.2, R8.2
- net at U1.3 (GAIN_ADJ_2): now also R4.2; no longer R2.2
- net CARRIER: now reaches C10.1, J3.1 (In)
- net OUT: now reaches C9.2, J2.1 (In)
- net OUT_A: now reaches C9.1
- net OUT_A: now also R9.2, U1.6 (OUT)
- net at U1.4 (SIG_IN): now also C1.1, R15.1, R16.1; no longer R4.2
- net MOD_A: now reaches U1.1 (SIG_IN_2)
- net MOD_A: now also C4.1, R14.1, R17.1
- net CARRIER_A: now reaches C10.2, R3.1, U1.10 (CARRIER_IN)
- net at U1.2 (GAIN_ADJ): now also R4.1
- net MOD: now reaches J4.1 (In)
- net MOD: now also C4.2
- new net: D2.2 (A), J5.1 (Pin_1)
- new net: R16.2, RV1.3
- new net: R12.1, U1.12 (OUT)
- new net: R14.2, R15.2, R6.1, R7.1
- new net: D3.2 (A), R2.2
- new net: R17.2, RV1.1
- new net V_IN: C5.1, C6.1, D2.1 (K), U3.1 (IN)
Other:
- moved on the sheet: C9, J2, R12, R4, R6, R7, R8
